File: Electronics/Source/mainboard.kicad_sch (KiCad schematic)
At the start: 22 parts, among them J1 Conn_01x03, J2 Conn_01x02, J3 Conn_01x02, J4 Conn_01x19_Socket, J5 Conn_01x19_Socket, SW1 Slide switch ON-ON, U1 L7805, U2 ESP32-DEVKITC, U3 L293

Commit message: STL transfers and kicad cleanup
Parts:
- R1, R2, R3, R4: value 330 ohm -> 1k
Connections:
- no-connect marks 27 -> 26
Other:
- note removed: "2x conn for motor 1x conn for battery 4x led (power, wifi, server, activity) 7805 voltage divider on-off switch ledler asagi bakacak konektorler iceride mumkunse kenarda onoff usb ile ayni tarafta"
- title: (none) -> Micro Invaders Driver Board
- moved on the sheet: C1, C2, D1, D2, D3, D4, F1, J1, J2, J3, J4, J5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
